File: modules_lpc1115/smokedetector/Rauchmelder.sch (EAGLE design)
At the start: 75 parts, among them IC1 BD9G101, IC2 LPC1115, Q1 BC856, Q3 BCP52, Q4 ASFL, T1 BC847C, T2 BC817

Commit message: [RM] - changed values to standard values
Parts:
- C103, C105: value 47uF/10V -> 47uF 10V
- C11, C8: value 10n -> 10nF
- L1: value 6.8µH -> 6.8uH
- renumbered C15 to C100, C16 to C103, C17 to C102, C21 to C101, C22 to C105, C7 to C104, D1 to D100, R10 to R101
Other:
- moved on the sheet: C20, D7, D8, FD1, FD2, FD3, FD4, LED1, R11, R13, R17, R19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
